File: Carte matrice/Carte matrice.kicad_sch (KiCad schematic)
At the start: 19 parts, among them SW1 SW_Push, SW2 SW_Push, SW3 SW_Push, SW4 SW_Push, SW5 SW_Push, SW6 SW_Push

Commit message: 30/01 BLE OK
BLE Connection ok caracteristique et service trouve faire envoi
Parts:
- removed D5, D6: LED, symbol Device:LED
- removed R1, R2: 1k, symbol Device:R
- removed R5: 100, symbol Device:R
- added D5, D6, D7, D8, D9: 1N4148, Diode_THT:D_DO-35_SOD27_P7.62mm_Horizontal, symbol Diode:1N4148
- added SW7, SW8, SW9: SW_Push, Button_Switch_THT:SW_Tactile_Straight_KSA0Axx1LFTR, symbol Switch:SW_Push
- R6: value 100 -> 10k
Connections:
- net Earth: no longer A1.D9
- net col 0: now also SW1.1, SW3.1, SW5.1; no longer SW2.1, SW4.1, SW6.1
- net col 1: now also SW2.1, SW4.1, SW6.1; no longer SW1.1, SW3.1, SW5.1
- net row 1: now also D7.1 (K)
- net row 2: now also D8.1 (K)
- net at SW5.2: now also D5.2 (A)
- net at SW6.2: now also D6.2 (A)
- net row 0: now reaches R6.2
- net row 0: now also A1.D9, D5.1 (K), D6.1 (K), D9.1 (K)
- new net: D8.2 (A), SW7.2
- new net: D7.2 (A), SW8.2
- new net: D9.2 (A), SW9.2
- new net col 2: SW7.1, SW8.1, SW9.1
Other:
- moved on the sheet: A1, D1, D2, D3, D4, R3, R4, SW1, SW2, SW3, SW4, SW5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

Commit message: Connection et envoie OK
Debut cahier de conception
Connection et envoie BLE OK
bouton reconnect OK
Faire envoie touches piano
Parts:
- removed R3, R4, R6: 10k, symbol Device:R
- added SW10, SW11, SW12, SW13: SW_Push, Button_Switch_THT:SW_Tactile_Straight_KSA0Axx1LFTR, symbol Switch:SW_Push
Connections:
- net row 0 is gone; now on net Earth: A1.D9, D5.1 (K), D6.1 (K), D9.1 (K)
- net row 1 is gone; now on net Earth: A1.D10, D3.1 (K), D4.1 (K), D7.1 (K)
- net row 2 is gone; now on net Earth: A1.D11 (D11_MOSI), D1.1 (K), D2.1 (K), D8.1 (K)
- net Earth: now also SW10.1, SW11.1, SW12.1, SW13.1
- new net Pin1: SW13.2
- new net Pin2: SW12.2
- new net Pin3: SW11.2
- new net Pin4: SW10.2
