File: PCB Symphonie/PCB Symphonie.kicad_pcb (KiCad board)
At the start: 2 copper layers, 129.1 x 84.7 mm, 41 parts, among them J1 Neopix Batt, J10 BTN, J11 Ligne Octave 1, J2 Neopix piano, J3 Alim ESP32, J4 Bornier Signal Ampli, J5 Conn_01x15_Pin, J6 Conn_01x15_Pin, J7 Colonne Octave 1, J8 Colonne Octave 2, J9 Ligne Octave 2

Commit message: Maj de bcp de truc
Parts:
- moved D23 4.13 mm to (165.1, 55.4)
- moved J6 1.02 mm to (183.4, 55.9)
Routing:
- net CA2: track 83.1 -> 104.6 mm, vias 0 -> 2
- net ROW4: track 78.8 -> 92.9 mm, vias 1 -> 3
- net CA: track 147.1 -> 135.7 mm
- net CB2: track 40.6 -> 51.2 mm, vias 0 -> 2
- net LED BLE: track 31.7 -> 40.2 mm
- net ROW3: track 92.3 -> 100.5 mm, vias 1 -> 2
- net +3.3V: track 112.4 -> 120.6 mm, vias 0 -> 3
- net CA#: track 82.5 -> 88.6 mm
- net ROW2: track 106.5 -> 111.4 mm, vias 1 -> 2
- net NEOPIX 1: track 20.8 -> 25.5 mm, vias 0 -> 1
- net CA#2: track 104.5 -> 107.5 mm
- net R_BTN: track 6.72 -> 9.07 mm
- net RC2: track 15.9 -> 14.4 mm
- net RB2: track 15.5 -> 14.1 mm
- net AMPLIFIER INPUT: track 48.6 -> 49.6 mm, vias 1 -> 0
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
Commit message: Carte elec
Parts:
- removed D0, D10, D11, D12, D13, D14, D15, D16, D17, D18, D19, D20, D21, D22, D23, D24, D8, D9: 1N4148, Diode_THT:D_DO-35_SOD27_P7.62mm_Horizontal
- removed D25, D26: LED, LED_THT:LED_D3.0mm
- removed R18, R19: R, Resistor_THT:R_Axial_DIN0204_L3.6mm_D1.6mm_P7.62mm_Horizontal
- added C1: 100n, Capacitor_THT:C_Rect_L7.0mm_W2.0mm_P5.00mm, F.Cu at (173.5, 50.5)
- added J12: 5V, TerminalBlock:TerminalBlock_MaiXu_MX126-5.0-02P_1x02_P5.00mm, F.Cu at (161.2, 39.1)
- added J13: Signal output, TerminalBlock:TerminalBlock_MaiXu_MX126-5.0-02P_1x02_P5.00mm, F.Cu at (173.5, 39.1)
- added R2: R, Resistor_THT:R_Axial_DIN0204_L3.6mm_D1.6mm_P7.62mm_Horizontal, F.Cu at (228.6, 45.8)
- added R3: R, Resistor_THT:R_Axial_DIN0204_L3.6mm_D1.6mm_P7.62mm_Horizontal, F.Cu at (234.4, 46.0)
- added R4: 47k, Resistor_THT:R_Axial_DIN0207_L6.3mm_D2.5mm_P7.62mm_Horizontal, F.Cu at (145.8, 65.0)
- added R5: 10k, Resistor_THT:R_Axial_DIN0207_L6.3mm_D2.5mm_P7.62mm_Horizontal, F.Cu at (145.8, 59.9)
- added R6: 33k, Resistor_THT:R_Axial_DIN0207_L6.3mm_D2.5mm_P7.62mm_Horizontal, F.Cu at (172.2, 46.2)
- added U1: TL081, Package_DIP:DIP-8_W7.62mm_Socket, F.Cu at (145.9, 48.5)
- added U2: TL081, Package_DIP:DIP-8_W7.62mm_Socket, F.Cu at (160.2, 48.5)
- D6, D7: value 1N4148 -> LED; footprint Diode_THT:D_DO-35_SOD27_P7.62mm_Horizontal -> LED_THT:LED_D3.0mm
- J1: value Neopix Batt -> Ligne Octave 2; footprint TerminalBlock:TerminalBlock_MaiXu_MX126-5.0-02P_1x02_P5.00mm -> Connector_PinSocket_2.54mm:PinSocket_1x12_P2.54mm_Vertical
- J10: value BTN -> Alim ESP32
- J11: value Ligne Octave 1 -> -5V; footprint Connector_PinSocket_2.54mm:PinSocket_1x12_P2.54mm_Vertical -> TerminalBlock:TerminalBlock_MaiXu_MX126-5.0-02P_1x02_P5.00mm
- J2: value Neopix piano -> Ligne Octave 1; footprint TerminalBlock:TerminalBlock_MaiXu_MX126-5.0-02P_1x02_P5.00mm -> Connector_PinSocket_2.54mm:PinSocket_1x12_P2.54mm_Vertical
- J3: value Alim ESP32 -> Neopix Batt
- J4: value Bornier Signal Ampli -> Neopix piano
- J7: value Colonne Octave 1 -> Colonne Octave 2
- J8: value Colonne Octave 2 -> Colonne Octave 1
- J9: value Ligne Octave 2 -> BTN; footprint Connector_PinSocket_2.54mm:PinSocket_1x12_P2.54mm_Vertical -> TerminalBlock:TerminalBlock_MaiXu_MX126-5.0-02P_1x02_P5.00mm
- moved J11 117.6 mm to (148.8, 39.1), turned to 0 degrees
- moved J1 106.6 mm to (139.9, 69.1)
- moved D1 85.5 mm to (146.8, 86.6)
- moved D5 84.9 mm to (146.8, 83.6)
- moved J4 82.8 mm to (236.0, 39.3), turned to 0 degrees
- moved R1 74.9 mm to (215.4, 45.7), turned to 180 degrees
- moved D7 66.5 mm to (165.9, 85.1)
- moved J9 43.1 mm to (136.1, 52.4), turned to -90 degrees
- moved J5 36.4 mm to (205.5, 92.2), turned to 180 degrees
- moved J6 36.4 mm to (180.6, 92.2), turned to 180 degrees
- moved J10 34.9 mm to (209.4, 39.1), turned to 0 degrees
- moved J2 34.8 mm to (250.2, 68.8)
- moved D6 24.4 mm to (224.8, 55.9)
- moved D4 15.8 mm to (242.1, 74.4), turned to 180 degrees
- moved D3 15.4 mm to (242.1, 78.5), turned to 180 degrees
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Connections:
- D1 pad 1: ROW0 -> RA#2
- D1 pad 2: RC# -> Net-(D1-A)
- D2 pad 1: ROW0 -> RA#
- D2 pad 2: RD -> Net-(D2-A)
- D3 pad 1: ROW0 -> RA
- D3 pad 2: RD# -> Net-(D3-A)
- D4 pad 1: ROW0 -> RC
- D4 pad 2: RE -> Net-(D4-A)
- D5 pad 1: ROW1 -> RD#2
- D5 pad 2: RF -> Net-(D5-A)
- D6 pad 1: ROW1 -> Net-(D6-K)
- D6 pad 2: RF# -> Earth
- D7 pad 1: ROW1 -> Earth
- D7 pad 2: RG -> LED BLE
- J1 pad 1: Net-(J1-Pin_1) -> RA#
- J1 pad 2: Earth -> RA#
- J10 pad 1: CA -> +3.3V
- J10 pad 2: R_BTN -> Earth
- J11 pad 1: RC -> Earth
- J11 pad 2: RC# -> -5V
- J2 pad 1: Net-(J2-Pin_1) -> RC
- J2 pad 2: Earth -> RC
- J3 pad 1: +3.3V -> Net-(J3-Pin_1)
- J4 pad 1: AMPLIFIER INPUT -> Net-(J4-Pin_1)
- J5 pad 1: NEOPIX 1 -> unconnected-(J5-Pin_1-Pad1)
- J5 pad 10: ROW0 -> CA2
- J5 pad 11: ROW3 -> CA#2
- J5 pad 12: unconnected-(J5-Pin_12-Pad12) -> CB2
- J5 pad 13: unconnected-(J5-Pin_13-Pad13) -> CA#
- J5 pad 15: +3.3V -> unconnected-(J5-Pin_15-Pad15)
- J5 pad 2: NEOPIX 2 -> BATT LVL INPUT
- J5 pad 5: LED BLE -> unconnected-(J5-Pin_5-Pad5)
- J5 pad 6: ROW4 -> unconnected-(J5-Pin_6-Pad6)
- J5 pad 7: ROW2 -> CA
- J5 pad 8: unconnected-(J5-Pin_8-Pad8) -> SIGNAL OUTPUT
- J5 pad 9: ROW1 -> unconnected-(J5-Pin_9-Pad9)
- J6 pad 1: Volume INPUT -> NEOPIX 1
- J6 pad 10: CA2 -> Net-(D4-A)
- J6 pad 11: CA#2 -> Net-(D5-A)
- J6 pad 12: CB2 -> unconnected-(J6-Pin_12-Pad12)
- J6 pad 13: CA# -> unconnected-(J6-Pin_13-Pad13)
- J6 pad 15: unconnected-(J6-Pin_15-Pad15) -> +3.3V
- J6 pad 2: BATT LVL INPUT -> NEOPIX 2
- J6 pad 5: unconnected-(J6-Pin_5-Pad5) -> LED BLE
- J6 pad 6: unconnected-(J6-Pin_6-Pad6) -> Net-(D1-A)
- J6 pad 7: CA -> Net-(D2-A)
- J6 pad 8: AMPLIFIER INPUT -> unconnected-(J6-Pin_8-Pad8)
- J6 pad 9: unconnected-(J6-Pin_9-Pad9) -> Net-(D3-A)
- J7 pad 1: CB2 -> CA#2
- J7 pad 10: CA# -> CB2
- J7 pad 11: CA#2 -> CB2
- J7 pad 12: CA#2 -> CB2
- J7 pad 2: CB2 -> CA#2
- J7 pad 3: CA2 -> CA#2
- J7 pad 4: CA2 -> CA#
- J7 pad 5: CA2 -> CA#
- J7 pad 8: CA# -> CA2
- J7 pad 9: CA# -> CA2
- J8 pad 1: CA#2 -> CB2
- J8 pad 10: CB2 -> CA#
- J8 pad 11: CB2 -> CA#2
- J8 pad 12: CB2 -> CA#2
- J8 pad 2: CA#2 -> CB2
- J8 pad 3: CA#2 -> CA2
- J8 pad 4: CA# -> CA2
- J8 pad 5: CA# -> CA2
- J8 pad 8: CA2 -> CA#
- J8 pad 9: CA2 -> CA#
- J9 pad 1: RC2 -> CA
- J9 pad 2: RC#2 -> RA#2
- R1 pad 1: Net-(D25-K) -> Net-(D6-K)
Routing:
- net RA#: track 15.0 -> 153.6 mm, vias 0 -> 2
- net ROW2: track 111.4 -> 0.00 mm, vias 2 -> 0
- net ROW3: track 100.5 -> 0.00 mm, vias 2 -> 0
- net SIGNAL OUTPUT: track 0.00 -> 99.5 mm, vias 0 -> 2
- net ROW4: track 92.9 -> 0.00 mm, vias 3 -> 0
- net Net-(D2-A): track 0.00 -> 86.0 mm
- net Net-(D4-A): track 0.00 -> 85.1 mm
- net Net-(D3-A): track 0.00 -> 84.4 mm
- net NEOPIX 1: track 25.5 -> 108.2 mm, vias 1 -> 2
- net +3.3V: track 120.6 -> 42.0 mm, vias 3 -> 0
- net NEOPIX 2: track 33.3 -> 108.6 mm, vias 1 -> 2
- net CB2: track 51.2 -> 126.3 mm
- net AMPLIFIER INPUT: track 49.6 -> 0.00 mm
- net -5V: track 0.00 -> 41.5 mm
- net CA: track 135.7 -> 176.6 mm, vias 0 -> 2
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- removed copper zone on B.Cu, net Earth
- removed copper zone on F.Cu, net Earth
Other:
- board text removed: "3V3"
- board text removed: "BTN"
- board text removed: "Ligne Octave 1"
- board text removed: "Ligne Octave 2"
- board text removed: "NEOPIX BATTERIE"
- board text removed: "NEOPIX PIANO"
- board text removed: "Sortie signal"
