File: PCB Symphonie/PCB Symphonie.kicad_sch (KiCad schematic)
At the start: 41 parts, among them J1 Neopix Batt, J10 BTN, J11 Ligne Octave 1, J2 Neopix piano, J3 Alim ESP32, J4 Bornier Signal Ampli, J5 Conn_01x15_Pin, J6 Conn_01x15_Pin, J7 Colonne Octave 1, J8 Colonne Octave 2, J9 Ligne Octave 2

Commit message: Carte elec
Parts:
- removed D0, D10, D11, D12, D13, D14, D15, D16, D17, D18, D19, D20, D21, D22, D23, D24, D6, D7, D8, D9: 1N4148, Diode_THT:D_DO-35_SOD27_P7.62mm_Horizontal, symbol Diode:1N4148
- removed J4: Bornier Signal Ampli, TerminalBlock:TerminalBlock_MaiXu_MX126-5.0-02P_1x02_P5.00mm, symbol Connector:Screw_Terminal_01x02
- added C1: 100n, Capacitor_THT:C_Rect_L7.0mm_W2.0mm_P5.00mm, symbol Device:C
- added J11: -5V, TerminalBlock:TerminalBlock_MaiXu_MX126-5.0-02P_1x02_P5.00mm, symbol Connector:Screw_Terminal_01x02
- added J12: 5V, TerminalBlock:TerminalBlock_MaiXu_MX126-5.0-02P_1x02_P5.00mm, symbol Connector:Screw_Terminal_01x02
- added J13: Signal output, TerminalBlock:TerminalBlock_MaiXu_MX126-5.0-02P_1x02_P5.00mm, symbol Connector:Screw_Terminal_01x02
- added R4: 47k, Resistor_THT:R_Axial_DIN0207_L6.3mm_D2.5mm_P7.62mm_Horizontal, symbol Device:R
- added R5: 10k, Resistor_THT:R_Axial_DIN0207_L6.3mm_D2.5mm_P7.62mm_Horizontal, symbol Device:R
- added R6: 33k, Resistor_THT:R_Axial_DIN0207_L6.3mm_D2.5mm_P7.62mm_Horizontal, symbol Device:R
- added U1, U2: TL081, Package_DIP:DIP-8_W7.62mm_Socket, symbol Amplifier_Operational:TL081
- renumbered D25 to D6, D26 to D7, J9 to J1, J3 to J10, J11 to J2, J1 to J3, J2 to J4, J6 to J5, J5 to J6, J8 to J7, J7 to J8, J10 to J9, R18 to R2, R19 to R3
Connections:
- net RA2 is gone; now on net RA#2: J1.10 (Pin_10)
- net RB is gone; now on net RA#: J2.12 (Pin_12)
- net RB2 is gone; now on net RA#2: J1.12 (Pin_12)
- net RC#2 is gone; now on net RA#: J1.2 (Pin_2)
- net RC2 is gone; now on net RA#: J1.1 (Pin_1)
- net RD2 is gone; now on net RA#: J1.3 (Pin_3)
- net RE2 is gone; now on net RD#2: J1.5 (Pin_5)
- net RF# is gone; now on net RA: J2.7 (Pin_7)
- net RF#2 is gone; now on net RD#2: J1.7 (Pin_7)
- net RF2 is gone; now on net RD#2: J1.6 (Pin_6)
- net RG is gone; now on net RA: J2.8 (Pin_8)
- net RG# is gone; now on net RA: J2.9 (Pin_9)
- net RG#2 is gone; now on net RA#2: J1.9 (Pin_9)
- net RG2 is gone; now on net RD#2: J1.8 (Pin_8)
- net ROW2 is gone; now on an unnamed net: J6.7 (Pin_7)
- net ROW3 is gone; now on an unnamed net: J6.11 (Pin_11)
- net ROW4 is gone; now on an unnamed net: J6.6 (Pin_6)
- net R_BTN is gone; now on net RA#2: J9.2 (Pin_2)
- net Earth: now also J11.1 (Pin_1), J12.1 (Pin_1), J13.1 (Pin_1), R6.1, U1.3 (+)
- net RA: now also D3.1 (K), J2.6 (Pin_6)
- net RA#: now also D2.1 (K)
- net RA#2: now also D1.1 (K)
- net RC: now also D4.1 (K), J2.2 (Pin_2), J2.3 (Pin_3), J2.4 (Pin_4), J2.5 (Pin_5)
- net RD#2: now also D5.1 (K)
- net AMPLIFIER INPUT renamed SIGNAL OUTPUT
- net SIGNAL OUTPUT: now also R4.2
- net RC#: no longer names the net of D1.2 (A)
- net RC#: no longer J2.2 (Pin_2)
- net RD: no longer names the net of D2.2 (A)
- net RD: no longer J2.3 (Pin_3)
- net RD#: no longer names the net of D3.2 (A)
- net RD#: now also J6.9 (Pin_9); no longer J2.4 (Pin_4)
- net RE: no longer names the net of D4.2 (A)
- net RE: now also J6.10 (Pin_10); no longer J2.5 (Pin_5)
- net RF: no longer names the net of D5.2 (A)
- net RF: no longer J2.6 (Pin_6)
- removed net ROW0: D1.1 (K), D2.1 (K), D3.1 (K), D4.1 (K), J6.10 (Pin_10)
- removed net ROW1: D5.1 (K), J6.9 (Pin_9)
- net Volume INPUT: no longer names the net of J5.1 (Pin_1)
- new net: C1.2, J13.2 (Pin_2), R6.2
- new net: C1.1, U2.2 (-), U2.6
- new net: R5.2, U1.6, U2.3 (+)
- new net: R4.1, R5.1, U1.2 (-)
- new net +5V: J12.2 (Pin_2), U1.7 (V+), U2.7 (V+)
- new net -5V: J11.2 (Pin_2), U1.4 (V-), U2.4 (V-)
Other:
- moved on the sheet: D6, D7, J10, J3, J4, J9, R1, R2, R3
